File: qspi-soc-pmod/qspi_soc_pmod/qspi_soc_pmod.kicad_pcb (KiCad board)
At the start: 4 copper layers, 66 x 22.5 mm, 27 parts, among them J1 Conn_02x06_Odd_Even, U1 74AHC138, U2 W25Q128JVS, U3 APS6404L-3SQR-SN, U4 APS6404L-3SQR-SN, U5 APS6404L-3SQR-SN, U6 APS6404L-3SQR-SN, U7 APS6404L-3SQR-SN, U8 APS6404L-3SQR-SN

Commit message: PCB update
Signed-off-by: gatecat <gatecat@ds0.me>
Parts:
- added J2: PROG, Connector_PinHeader_2.54mm:PinHeader_1x05_P2.54mm_Vertical, F.Cu at (61.6, 91.0)
- added J3: MODE, Connector_PinHeader_2.54mm:PinHeader_1x03_P2.54mm_Vertical, F.Cu at (66.0, 73.0)
- added R11: 10k, Resistor_SMD:R_0603_1608Metric, F.Cu at (114.2, 87.0)
- added R12: 10k, Resistor_SMD:R_0603_1608Metric, F.Cu at (114.2, 91.0)
Connections:
- U1 pad 15: /FLASH_CSN -> /FLASH_CSN_SOC
Routing:
- net /PROG_CSN: track 0.00 -> 23.5 mm
- net /QSPI_CLK: track 111.9 -> 133.8 mm
- net /QSPI_D0: track 113.4 -> 133.4 mm
- net +3V3: track 51.7 -> 71.2 mm
- net /QSPI_D1: track 119.6 -> 136.0 mm
- net /FLASH_CSN_SOC: track 0.00 -> 14.3 mm
- net /FLASH_CSN: track 12.5 -> 18.4 mm, vias 0 -> 1
- net /QSPI_D2: track 116.4 -> 121.1 mm
- net /QSPI_D3: track 115.5 -> 117.0 mm
Other:
- board text added: "P"
- board text added: "R"
