File: qspi-soc-pmod/qspi_soc_pmod/qspi_soc_pmod.kicad_sch (KiCad schematic)
At the start: 27 parts, among them J1 Conn_02x06_Top_Bottom, U1 74AHC138, U2 W25Q128JVS, U3 APS6404L-3SQR-SN, U4 APS6404L-3SQR-SN, U5 APS6404L-3SQR-SN, U6 APS6404L-3SQR-SN, U7 APS6404L-3SQR-SN, U8 APS6404L-3SQR-SN

Commit message: QSPI PMOD PCB
Signed-off-by: gatecat <gatecat@ds0.me>
Parts:
- J1: value Conn_02x06_Top_Bottom -> Conn_02x06_Odd_Even; footprint Resistor_SMD:R_0603_1608Metric -> Connector_PinHeader_2.54mm:PinHeader_2x06_P2.54mm_Horizontal; symbol Connector_Generic:Conn_02x06_Top_Bottom -> Connector_Generic:Conn_02x06_Odd_Even
Connections:
- net +3V3: now also J1.2 (Pin_2); no longer J1.7 (Pin_7)
- net GND: now also J1.3 (Pin_3), J1.4 (Pin_4); no longer J1.2 (Pin_2), J1.8 (Pin_8)
- net QSPI_A0: now also J1.8 (Pin_8); no longer J1.5 (Pin_5)
- net QSPI_A1: now also J1.5 (Pin_5); no longer J1.6 (Pin_6)
- net QSPI_A2: now also J1.6 (Pin_6); no longer J1.12 (Pin_12)
- net QSPI_CLK: now also J1.9 (Pin_9); no longer J1.11 (Pin_11)
- net QSPI_D0: now also J1.7 (Pin_7); no longer J1.9 (Pin_9)
- net QSPI_D1: now also J1.12 (Pin_12); no longer J1.3 (Pin_3)
- net QSPI_D2: now also J1.10 (Pin_10); no longer J1.4 (Pin_4)
- net QSPI_D3: now also J1.11 (Pin_11); no longer J1.10 (Pin_10)
Changed lines of the file:
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@@
     (effects (font (size 1.27 1.27)) (justify left bottom))
   )
-  (label "QSPI_A2" (at 17.78 44.45 0)
+  (label "QSPI_D1" (at 17.78 44.45 0)
     (effects (font (size 1.27 1.27)) (justify left bottom))
   )
@@
     (effects (font (size 1.27 1.27)) (justify right bottom))
   )
-  (label "QSPI_CLK" (at 17.78 41.91 0)
+  (label "QSPI_D2" (at 17.78 41.91 0)
     (effects (font (size 1.27 1.27)) (justify left bottom))
   )
@@
     (effects (font (size 1.27 1.27)) (justify left bottom))
   )
-  (label "QSPI_D2" (at 71.12 39.37 180)
-    (effects (font (size 1.27 1.27)) (justify right bottom))
-  )
-  (label "QSPI_A0" (at 71.12 41.91 180)
+  (label "QSPI_D0" (at 71.12 39.37 180)
+    (effects (font (size 1.27 1.27)) (justify right bottom))
+  )
+  (label "QSPI_CLK" (at 71.12 41.91 180)
     (effects (font (size 1.27 1.27)) (justify right bottom))
   )
@@
     (effects (font (size 1.27 1.27)) (justify left bottom))
   )
-  (label "QSPI_D3" (at 17.78 39.37 0)
+  (label "QSPI_A0" (at 17.78 39.37 0)
     (effects (font (size 1.27 1.27)) (justify left bottom))
   )
@@
     (effects (font (size 1.27 1.27)) (justify right bottom))
   )
-  (label "QSPI_A1" (at 71.12 44.45 180)
+  (label "QSPI_D3" (at 71.12 44.45 180)
     (effects (font (size 1.27 1.27)) (justify right bottom))
   )
@@
     (effects (font (size 1.27 1.27)) (justify right bottom))
   )
-  (label "QSPI_D1" (at 71.12 36.83 180)
+  (label "QSPI_A1" (at 71.12 36.83 180)
     (effects (font (size 1.27 1.27)) (justify right bottom))
   )
@@
     (effects (font (size 1.27 1.27)) (justify right bottom))
   )
-  (label "QSPI_D0" (at 17.78 36.83 0)
+  (label "QSPI_A2" (at 17.78 36.83 0)
     (effects (font (size 1.27 1.27)) (justify left bottom))
   )
@@
     (pin "1")
   )
-  (symbol (lib_id "Connector_Generic:Conn_02x06_Top_Bottom") (at 45.72 36.83 0) (mirror y) (unit 1)
+  (symbol (lib_id "Connector_Generic:Conn_02x06_Odd_Even") (at 45.72 36.83 0) (mirror y) (unit 1)
     (in_bom yes) (on_board yes) (fields_autoplaced)
     (property "Reference" "J1" (id 0) (at 44.45 25.4 0))
-    (property "Value" "Conn_02x06_Top_Bottom" (id 1) (at 44.45 27.94 0))
-    (property "Footprint" "Resistor_SMD:R_0603_1608Metric" (id 2) (at 45.72 36.83 0)
+    (property "Value" "Conn_02x06_Odd_Even" (id 1) (at 44.45 46.99 0))
+    (property "Footprint" "Connector_PinHeader_2.54mm:PinHeader_2x06_P2.54mm_Horizontal" (id 2) (at 45.72 36.83 0)
       (effects (font (size 1.27 1.27)) hide)
     )
@@
     )
     (path "/f1cc6dfb-a376-4360-b675-90fd280cc969"
-      (reference "J1") (unit 1) (value "Conn_02x06_Top_Bottom") (footprint "Resistor_SMD:R_0603_1608Metric")
+      (reference "J1") (unit 1) (value "Conn_02x06_Odd_Even") (footprint "Connector_PinHeader_2.54mm:PinHeader_2x06_P2.54mm_Horizontal")
     )
     (path "/a2a75006-b0fd-4df5-a0db-6005c4dfb1f0"

Commit message: PCB update
Signed-off-by: gatecat <gatecat@ds0.me>
Parts:
- added J2: PROG, Connector_PinHeader_2.54mm:PinHeader_1x05_P2.54mm_Vertical, symbol Connector_Generic:Conn_01x05
- added J3: MODE, Connector_PinHeader_2.54mm:PinHeader_1x03_P2.54mm_Vertical, symbol Connector_Generic:Conn_01x03
- added R11, R12: 10k, Resistor_SMD:R_0603_1608Metric, symbol Device:R_Small
Connections:
- net +3V3: now also R11.2, R12.2
- net FLASH_CSN: now also J3.2 (Pin_2); no longer U1.15 (~{Y0})
- net GND: now also J2.5 (Pin_5)
- net QSPI_CLK: now also J2.2 (Pin_2)
- net QSPI_D0: now also J2.3 (Pin_3)
- net QSPI_D1: now also J2.1 (Pin_1)
- net QSPI_D2: now also R12.1
- net QSPI_D3: now also R11.1
- new net FLASH_CSN_SOC: J3.1 (Pin_1), U1.15 (~{Y0})
- new net PROG_CSN: J2.4 (Pin_4), J3.3 (Pin_3)
